Commit message: Robot path planning in static enviromet

File: ur3_description/urdf/ur3.urdf (robot description, URDF)
Before this commit: robot ur3_workplace, 28 links, 27 joints
Links:
- added link back_wall; collision box size=0.75 0.1 1.2
- added link left_wall; collision box size=0.1 0.9 1.2
- added link top_wall; collision box size=0.75 0.9 0.1
- link effector_body: geometry collision mesh filename=package://ur3_description/meshes/effector_body.stl scale=0.001 0.001 0.001; visual mesh filename=package://ur3_description/meshes/effector_body.stl scale=0.001 0.001 0.001
- link force_sensor: geometry collision mesh filename=package://ur3_description/meshes/force_sensor.stl scale=0.001 0.001 0.001; visual mesh filename=package://ur3_description/meshes/force_sensor.stl scale=0.001 0.001 0.001
- link left_jaw: geometry collision mesh filename=package://ur3_description/meshes/jaw.stl scale=0.001 0.001 0.001; visual mesh filename=package://ur3_description/meshes/jaw.stl scale=0.001 0.001 0.001
- link right_jaw: geometry collision mesh filename=package://ur3_description/meshes/jaw.stl scale=0.001 0.001 0.001; visual mesh filename=package://ur3_description/meshes/jaw.stl scale=0.001 0.001 0.001
Joints:
- added joint back_wall_joint: type fixed, parent table, child back_wall, origin xyz=0.2 -0.32 0.1 rpy=0 0 0
- added joint left_wall_joint: type fixed, parent table, child left_wall, origin xyz=-0.22 0.18 0.1 rpy=0 0 0
- added joint top_wall_joint: type fixed, parent table, child top_wall, origin xyz=0.2 0.18 0.75 rpy=0 0 0
- joint leftjaw_to_effector: origin xyz=0 -0.01 0.076 rpy=0 0 0 -> xyz=0 0 0.076 rpy=0 0 0
- joint rightjaw_to_effector: origin xyz=0 0.01 0.076 rpy=0 0 3.14159265359 -> xyz=0 0 0.076 rpy=0 0 3.14159265359

File: ur3_description/urdf/ur3.xacro (robot description, xacro)
@@ -91,6 +91,7 @@
     <collision>
       <geometry>
-        <cylinder radius="0.035" length="0.035"/>
-      </geometry>
+        <mesh filename="package://ur3_description/meshes/force_sensor.stl" scale="0.001 0.001 0.001"/>
+      </geometry>
+      <origin rpy="${pi/2} 0 0" xyz="0 0 0"/>
     </collision>
   </link>
@@ -107,6 +108,7 @@
     <collision>
       <geometry>
-        <cylinder radius="0.031" length="0.076"/>
-      </geometry>
+        <mesh filename="package://ur3_description/meshes/effector_body.stl" scale="0.001 0.001 0.001"/>
+      </geometry>
+      <origin rpy="${pi/2} 0 0" xyz="0 0 0"/>
     </collision>
   </link>
@@ -123,6 +125,8 @@
     <collision>
       <geometry>
-        <box size="0.03 0.03 0.045"/>
-      </geometry>
+        <mesh filename="package://ur3_description/meshes/jaw.stl" scale="0.001 0.001 0.001"/>
+        <!-- <box size="0.03 0.03 0.045"/> -->
+      </geometry>
+      <origin rpy="${pi} 0 ${pi/2}" xyz="0 0 0"/>
     </collision>
   </link>
@@ -139,6 +143,8 @@
     <collision>
       <geometry>
-        <box size="0.03 0.03 0.045"/>
-      </geometry>
+        <!-- <box size="0.03 0.03 0.045"/> -->
+        <mesh filename="package://ur3_description/meshes/jaw.stl" scale="0.001 0.001 0.001"/>
+      </geometry>
+       <origin rpy="${pi} 0 ${pi/2}" xyz="0 0 0"/>
     </collision>
   </link>
@@ -159,5 +165,5 @@
     <parent link="effector_body"/>
     <child link="left_jaw"/>
-    <origin xyz="0 -0.01 0.076" rpy="0 0 0"/>
+    <origin xyz="0 0 0.076" rpy="0 0 0"/>
   </joint>
   <!--<joint name="rightjaw_to_effector" type="prismatic">-->
@@ -167,5 +173,5 @@
     <parent link="effector_body"/>
     <child link="right_jaw"/>
-    <origin xyz="0 0.01 0.076" rpy="0 0 ${pi}"/>
+    <origin xyz="0 0 0.076" rpy="0 0 ${pi}"/>
   </joint>
   <link name="camera_points_link"/>
@@ -175,3 +181,65 @@
     <child link="camera_points_link"/>
   </joint>
+  <xacro:property name="top_wall_z" value="0.75" />
+  <xacro:property name="limit_wall_height" value="${top_wall_z + 0.45}" />
+  <link name="top_wall">
+    <!-- <visual>
+      <geometry>
+        <box size="0.75 0.9 0.1"/>
+      </geometry>
+      <material name="black">
+        <color rgba="0 0 0 1" />
+      </material>
+    </visual> -->
+    <collision>
+      <geometry>
+        <box size="0.75 0.9 0.1"/>
+      </geometry>
+    </collision>
+  </link>
+  <joint name="top_wall_joint" type="fixed">
+    <origin rpy="0 0 0" xyz="0.2 0.18 ${top_wall_z}"/>
+    <parent link="table"/>
+    <child link="top_wall"/>
+  </joint>
+    <link name="back_wall">
+    <!-- <visual>
+      <geometry>
+        <box size="0.75 0.1 ${limit_wall_height}"/>
+      </geometry>
+      <material name="black">
+        <color rgba="0 0 0 1" />
+      </material>
+    </visual> -->
+    <collision>
+      <geometry>
+         <box size="0.75 0.1 ${limit_wall_height}"/>
+      </geometry>
+    </collision>
+  </link>
+  <joint name="back_wall_joint" type="fixed">
+    <origin rpy="0 0 0" xyz="0.2 -0.32 0.1"/>
+    <parent link="table"/>
+    <child link="back_wall"/>
+  </joint>
+    <link name="left_wall">
+    <!-- <visual>
+      <geometry>
+        <box size="0.1 0.9 ${limit_wall_height}"/>
+      </geometry>
+      <material name="black">
+        <color rgba="0 0 0 1" />
+      </material>
+    </visual> -->
+    <collision>
+      <geometry>
+         <box size="0.1 0.9 ${limit_wall_height}"/>
+      </geometry>
+    </collision>
+  </link>
+  <joint name="left_wall_joint" type="fixed">
+    <origin rpy="0 0 0" xyz="-0.22 0.18 0.1"/>
+    <parent link="table"/>
+    <child link="left_wall"/>
+  </joint>
 </robot>
