Commit message: ur3_multicam.xacro - is the version with two cameras

File: ur3_description/urdf/ur3.xacro (robot description, xacro)
@@ -5,5 +5,9 @@
   <xacro:include filename="$(find ur3_description)/urdf/depth_camera.xacro" />
   <depth_camera name="camera" />
-  <depth_camera name="camera2" />
+  <joint name="table_to_camera" type="fixed">
+    <parent link="table"/>
+    <child link="base_link_camera"/>
+    <origin xyz="0.165 0.94 0.55" rpy="0 ${pi/6} -${pi/2}"/>
+  </joint>
   <link name="world" />
   <link name="table">
@@ -33,14 +37,4 @@
     <child link="base_link"/>
     <origin xyz="0 0 0" rpy="0 0 0"/>
-  </joint>
-  <joint name="table_to_camera" type="fixed">
-    <parent link="table"/>
-    <child link="base_link_camera"/>
-    <origin xyz="0.165 0.94 0.55" rpy="0 ${pi/6} -${pi/2}"/>
-  </joint>
-  <joint name="table_to_camera2" type="fixed">
-    <parent link="table"/>
-    <child link="base_link_camera2"/>
-    <origin xyz="0.94 0.165 0.55" rpy="0 ${pi/6} -${pi}"/>
   </joint>
   <link name="force_sensor">
@@ -111,5 +105,5 @@
         <mesh filename="package://ur3_description/meshes/jaw.stl" scale="0.001 0.001 0.001"/>
       </geometry>
-       <origin rpy="${pi} 0 ${pi/2}" xyz="0 0 0"/>
+      <origin rpy="${pi} 0 ${pi/2}" xyz="0 0 0"/>
     </collision>
   </link>

File: ur3_description/urdf/ur3_multicam.xacro (robot description, xacro)
@@ -1,251 +1,10 @@
-<?xml version="1.0" ?>
 <robot name="ur3_workplace"
   xmlns:xacro="http://www.ros.org/wiki/xacro">
-  <xacro:include filename="$(find ur3_description)/urdf/ur3_robot_custom.urdf.xacro" />
-  <xacro:include filename="$(find ur3_description)/urdf/d435_camera_custom.urdf.xacro" />
-  <gazebo reference="camera_color_frame">
-    <sensor name="camera" type="depth">
-      <update_rate>20</update_rate>
-      <camera>
-        <horizontal_fov>1.047198</horizontal_fov>
-        <image>
-          <width>640</width>
-          <height>480</height>
-          <format>R8G8B8</format>
-        </image>
-        <clip>
-          <near>0.05</near>
-          <far>3</far>
-        </clip>
-      </camera>
-      <plugin name="camera_plugin" filename="libgazebo_ros_openni_kinect.so">
-        <baseline>0</baseline>
-        <alwaysOn>true</alwaysOn>
-        <!-- Keep this zero, update_rate in the parent <sensor> tag will control the frame rate. -->
-        <updateRate>0.0</updateRate>
-        <cameraName>camera_ir</cameraName>
-        <imageTopicName>/camera/color/image_raw</imageTopicName>
-        <cameraInfoTopicName>/camera/color/camera_info</cameraInfoTopicName>
-        <depthImageTopicName>/camera/depth/image_raw</depthImageTopicName>
-        <depthImageCameraInfoTopicName>/camera/depth/camera_info</depthImageCameraInfoTopicName>
-        <pointCloudTopicName>/camera/depth/color/points</pointCloudTopicName>
-        <frameName>camera_color_optical_frame</frameName>
-        <pointCloudCutoff>0.001</pointCloudCutoff>
-        <pointCloudCutoffMax>1.8</pointCloudCutoffMax>
-        <distortionK1>0</distortionK1>
-        <distortionK2>0</distortionK2>
-        <distortionK3>0</distortionK3>
-        <distortionT1>0</distortionT1>
-        <distortionT2>0</distortionT2>
-        <CxPrime>0</CxPrime>
-        <Cx>0</Cx>
-        <Cy>0</Cy>
-        <focalLength>0</focalLength>
-        <hackBaseline>0</hackBaseline>
-      </plugin>
-    </sensor>
-  </gazebo>
-  <link name="cam2" />
-  <joint name="world_to_cam" type="fixed">
-    <parent link="world"/>
-    <child link="cam2"/>
-    <origin xyz="0.94 -0.165 1.16" rpy="0 ${pi/6} 0"/>
-  </joint>
-  <link name="world" />
-  <link name="table">
-    <visual>
-      <geometry>
-        <mesh filename="package://ur3_description/meshes/stul.stl" scale="0.001 0.001 0.001"/>
-      </geometry>
-      <origin rpy="0 ${-pi/2} 0" xyz="0.47 -0.18 -0.51"/>
-      <material name="grey">
-        <color rgba="0.5 0.5 0.5 1" />
-      </material>
-    </visual>
-    <collision>
-      <geometry>
-        <box size="0.56 0.76 0.6"/>
-      </geometry>
-      <origin rpy="0 0 0" xyz="0.205 0.185 -0.295"/>
-    </collision>
-  </link>
-  <joint name="world_to_table" type="fixed">
-    <parent link="world"/>
-    <child link="table"/>
-    <origin xyz="0 0 0.61" rpy="0 0 0"/>
-  </joint>
-  <joint name="table_to_robot" type="fixed">
+  <xacro:include filename="$(find ur3_description)/urdf/ur3.xacro" />
+  <depth_camera name="camera2" />
+  <joint name="table_to_camera2" type="fixed">
     <parent link="table"/>
-    <child link="base_link"/>
-    <origin xyz="0 0 0" rpy="0 0 0"/>
-  </joint>
-  <joint name="table_to_camera" type="fixed">
-    <parent link="table"/>
-    <child link="base_link_camera"/>
-    <origin xyz="0.165 0.94 0.55" rpy="0 ${pi/6} -${pi/2}"/>
-  </joint>
-  <link name="force_sensor">
-    <visual>
-      <geometry>
-        <mesh filename="package://ur3_description/meshes/force_sensor.stl" scale="0.001 0.001 0.001"/>
-      </geometry>
-      <material name="grey">
-        <color rgba="0.5 0.5 0.5 1" />
-      </material>
-      <origin rpy="${pi/2} 0 0" xyz="0 0 0"/>
-    </visual>
-    <collision>
-      <geometry>
-        <mesh filename="package://ur3_description/meshes/force_sensor.stl" scale="0.001 0.001 0.001"/>
-      </geometry>
-      <origin rpy="${pi/2} 0 0" xyz="0 0 0"/>
-    </collision>
-  </link>
-  <link name="effector_body">
-    <visual>
-      <geometry>
-        <mesh filename="package://ur3_description/meshes/effector_body.stl" scale="0.001 0.001 0.001"/>
-      </geometry>
-      <material name="red">
-        <color rgba="1 0 0 1" />
-      </material>
-      <origin rpy="${pi/2} 0 0" xyz="0 0 0"/>
-    </visual>
-    <collision>
-      <geometry>
-        <mesh filename="package://ur3_description/meshes/effector_body.stl" scale="0.001 0.001 0.001"/>
-      </geometry>
-      <origin rpy="${pi/2} 0 0" xyz="0 0 0"/>
-    </collision>
-  </link>
-  <link name="left_jaw">
-    <visual>
-      <geometry>
-        <mesh filename="package://ur3_description/meshes/jaw.stl" scale="0.001 0.001 0.001"/>
-      </geometry>
-      <material name="black">
-        <color rgba="0 0 0 1" />
-      </material>
-      <origin rpy="${pi} 0 ${pi/2}" xyz="0 0 0"/>
-    </visual>
-    <collision>
-      <geometry>
-        <mesh filename="package://ur3_description/meshes/jaw.stl" scale="0.001 0.001 0.001"/>
-        <!-- <box size="0.03 0.03 0.045"/> -->
-      </geometry>
-      <origin rpy="${pi} 0 ${pi/2}" xyz="0 0 0"/>
-    </collision>
-  </link>
-  <link name="right_jaw">
-    <visual>
-      <geometry>
-        <mesh filename="package://ur3_description/meshes/jaw.stl" scale="0.001 0.001 0.001"/>
-      </geometry>
-      <material name="black">
-        <color rgba="0 0 0 1" />
-      </material>
-      <origin rpy="${pi} 0 ${pi/2}" xyz="0 0 0"/>
-    </visual>
-    <collision>
-      <geometry>
-        <!-- <box size="0.03 0.03 0.045"/> -->
-        <mesh filename="package://ur3_description/meshes/jaw.stl" scale="0.001 0.001 0.001"/>
-      </geometry>
-       <origin rpy="${pi} 0 ${pi/2}" xyz="0 0 0"/>
-    </collision>
-  </link>
-  <joint name="FT_to_tip" type="fixed">
-    <parent link="ee_link"/>
-    <child link="force_sensor"/>
-    <origin xyz="0 0 0" rpy="0 ${pi/2} 0"/>
-  </joint>
-  <joint name="Effector_to_FT" type="fixed">
-    <parent link="force_sensor"/>
-    <child link="effector_body"/>
-    <origin xyz="0 0 0.035" rpy="0 0 0"/>
-  </joint>
-  <!--<joint name="leftjaw_to_effector" type="prismatic">-->
-  <joint name="leftjaw_to_effector" type="fixed">
-    <!--  <axis xyz="0 1 0"/>
-  <limit effort="1000.0" lower="0.01" upper="0" velocity="0.5"/>-->
-    <parent link="effector_body"/>
-    <child link="left_jaw"/>
-    <origin xyz="0 0 0.076" rpy="0 0 0"/>
-  </joint>
-  <!--<joint name="rightjaw_to_effector" type="prismatic">-->
-  <joint name="rightjaw_to_effector" type="fixed">
-    <!--  <axis xyz="0 1 0"/>
-  <limit effort="1000.0" lower="0.01" upper="0" velocity="0.5"/> -->
-    <parent link="effector_body"/>
-    <child link="right_jaw"/>
-    <origin xyz="0 0 0.076" rpy="0 0 ${pi}"/>
-  </joint>
-  <link name="camera_points_link"/>
-  <joint name="camera_points_joint" type="fixed">
-    <origin rpy="0 1.57 0" xyz="0 0 0"/>
-    <parent link="base_link_camera"/>
-    <child link="camera_points_link"/>
-  </joint>
-  <xacro:property name="top_wall_z" value="0.75" />
-  <xacro:property name="limit_wall_height" value="${top_wall_z + 0.45}" />
-  <link name="top_wall">
-    <!-- <visual>
-      <geometry>
-        <box size="0.75 0.9 0.1"/>
-      </geometry>
-      <material name="black">
-        <color rgba="0 0 0 1" />
-      </material>
-    </visual> -->
-    <collision>
-      <geometry>
-        <box size="0.75 0.9 0.1"/>
-      </geometry>
-    </collision>
-  </link>
-  <joint name="top_wall_joint" type="fixed">
-    <origin rpy="0 0 0" xyz="0.2 0.18 ${top_wall_z}"/>
-    <parent link="table"/>
-    <child link="top_wall"/>
-  </joint>
-    <link name="back_wall">
-    <!-- <visual>
-      <geometry>
-        <box size="0.75 0.1 ${limit_wall_height}"/>
-      </geometry>
-      <material name="black">
-        <color rgba="0 0 0 1" />
-      </material>
-    </visual> -->
-    <collision>
-      <geometry>
-         <box size="0.75 0.1 ${limit_wall_height}"/>
-      </geometry>
-    </collision>
-  </link>
-  <joint name="back_wall_joint" type="fixed">
-    <origin rpy="0 0 0" xyz="0.2 -0.32 0.1"/>
-    <parent link="table"/>
-    <child link="back_wall"/>
-  </joint>
-    <link name="left_wall">
-    <!-- <visual>
-      <geometry>
-        <box size="0.1 0.9 ${limit_wall_height}"/>
-      </geometry>
-      <material name="black">
-        <color rgba="0 0 0 1" />
-      </material>
-    </visual> -->
-    <collision>
-      <geometry>
-         <box size="0.1 0.9 ${limit_wall_height}"/>
-      </geometry>
-    </collision>
-  </link>
-  <joint name="left_wall_joint" type="fixed">
-    <origin rpy="0 0 0" xyz="-0.22 0.18 0.1"/>
-    <parent link="table"/>
-    <child link="left_wall"/>
+    <child link="base_link_camera2"/>
+    <origin xyz="0.94 0.165 0.55" rpy="0 ${pi/6} -${pi}"/>
   </joint>
 </robot>

File: ur3_description/urdf/ur3_workspace_limitation.xacro (robot description, xacro)
@@ -11,5 +11,5 @@
       </geometry>
       <material name="black">
-        <color rgba="0 0 0 1" />
+        <color rgba="0.2 0.2 0.2 0.2" />
       </material>
     </visual> -->
@@ -31,5 +31,5 @@
       </geometry>
       <material name="black">
-        <color rgba="0 0 0 1" />
+        <color rgba="0.2 0.2 0.2 0.2" />
       </material>
     </visual> -->
@@ -51,5 +51,5 @@
       </geometry>
       <material name="black">
-        <color rgba="0 0 0 1" />
+        <color rgba="0.2 0.2 0.2 0.2" />
       </material>
     </visual> -->

Commit message: New xacro workspace

File: ur3_description/urdf/ur3.xacro (robot description, xacro)
@@ -8,5 +8,5 @@
     <parent link="table"/>
     <child link="base_link_camera"/>
-    <origin xyz="0.165 0.94 0.55" rpy="0 ${pi/6} -${pi/2}"/>
+    <origin xyz="-0.4 1.4 1.6" rpy="0 ${pi/6} -${pi/2}"/>
   </joint>
   <link name="world" />
@@ -14,7 +14,7 @@
     <visual>
       <geometry>
-        <mesh filename="package://ur3_description/meshes/stul.stl" scale="0.001 0.001 0.001"/>
+        <mesh filename="package://ur3_description/meshes/table.stl" scale="0.001 0.001 0.001"/>
       </geometry>
-      <origin rpy="0 ${-pi/2} 0" xyz="0.47 -0.18 -0.51"/>
+      <origin rpy="0 ${-pi/2} 0" xyz="0.0 0.0 0.0"/>
       <material name="grey">
         <color rgba="0.5 0.5 0.5 1" />
@@ -23,18 +23,57 @@
     <collision>
       <geometry>
-        <box size="0.56 0.76 0.6"/>
+        <mesh filename="package://ur3_description/meshes/table_collision.stl" scale="0.001 0.001 0.001"/>
       </geometry>
-      <origin rpy="0 0 0" xyz="0.205 0.185 -0.295"/>
+      <origin rpy="0 ${-pi/2} 0" xyz="0 0 0 "/>
     </collision>
   </link>
+  <link name="table_left_sup">
+    <collision>
+      <geometry>
+        <mesh filename="package://ur3_description/meshes/table_left_sup.stl" scale="0.001 0.001 0.001"/>
+      </geometry>
+      <origin rpy="0 ${-pi/2} 0" xyz="0 0 0 "/>
+    </collision>
+  </link>
+  <joint name="table_left_sup_j" type="fixed">
+    <parent link="table"/>
+    <child link="table_left_sup"/>
+    <origin xyz="0 0 0" rpy="0 0 0"/>
+  </joint>
+    <link name="table_right_sup">
+    <collision>
+      <geometry>
+        <mesh filename="package://ur3_description/meshes/table_right_sup.stl" scale="0.001 0.001 0.001"/>
+      </geometry>
+      <origin rpy="0 ${-pi/2} 0" xyz="0 0 0 "/>
+    </collision>
+  </link>
+  <joint name="table_right_sup_j" type="fixed">
+    <parent link="table"/>
+    <child link="table_right_sup"/>
+    <origin xyz="0 0 0" rpy="0 0 0"/>
+  </joint>
+  <link name="table_back_sup">
+    <collision>
+      <geometry>
+        <mesh filename="package://ur3_description/meshes/table_back_sup.stl" scale="0.001 0.001 0.001"/>
+      </geometry>
+      <origin rpy="0 ${-pi/2} 0" xyz="0 0 0 "/>
+    </collision>
+  </link>
+  <joint name="table_back_sup_j" type="fixed">
+    <parent link="table"/>
+    <child link="table_back_sup"/>
+    <origin xyz="0 0 0" rpy="0 0 0"/>
+  </joint>
   <joint name="world_to_table" type="fixed">
     <parent link="world"/>
     <child link="table"/>
-    <origin xyz="0 0 0.61" rpy="0 0 0"/>
+    <origin xyz="1 0 0" rpy="0 0 0"/>
   </joint>
   <joint name="table_to_robot" type="fixed">
     <parent link="table"/>
     <child link="base_link"/>
-    <origin xyz="0 0 0" rpy="0 0 0"/>
+    <origin xyz="-0.58 0.49 0.972" rpy="0 0 0"/>
   </joint>
   <link name="force_sensor">

File: ur3_description/urdf/ur3_multicam.xacro (robot description, xacro)
@@ -1,10 +1,10 @@
 <robot name="ur3_workplacess"
   xmlns:xacro="http://www.ros.org/wiki/xacro">
-  <xacro:include filename="$(find ur3_description)/urdf/ur3_workspace_limitation.xacro" />
+  <xacro:include filename="$(find ur3_description)/urdf/ur3.xacro" />
   <depth_camera name="camera2" />
   <joint name="table_to_camera2" type="fixed">
     <parent link="table"/>
     <child link="base_link_camera2"/>
-    <origin xyz="0.94 0.165 0.55" rpy="0 ${pi/6} -${pi}"/>
+    <origin xyz="0.1 0.5 1.4"  rpy="0 ${pi/6} -${pi}"/>
   </joint>
   <depth_camera name="camera_top" />
@@ -12,5 +12,5 @@
     <parent link="table"/>
     <child link="base_link_camera_top"/>
-    <origin xyz="0.2 0.185 1.2" rpy="0 ${pi/2} -${pi}"/>
+    <origin xyz="-0.4 0.5 2.1"  rpy="0 ${pi/2} -${pi}"/>
   </joint>
 </robot>

File: ur3_description/urdf/ur3_robot_custom.urdf.xacro (robot description, xacro)
@@ -2,6 +2,6 @@
 <robot xmlns:xacro="http://wiki.ros.org/xacro" name="ur3">
   <xacro:arg name="transmission_hw_interface" default="hardware_interface/PositionJointInterface"/>
-  <xacro:include filename="$(find ur_description)/urdf/common.gazebo.xacro" />
-  <xacro:include filename="$(find ur_description)/urdf/ur3.urdf.xacro" />
-  <xacro:ur3_robot prefix="" joint_limited="false" transmission_hw_interface="$(arg transmission_hw_interface)" />
+  <xacro:include filename="$(find ur_e_description)/urdf/common.gazebo.xacro" />
+  <xacro:include filename="$(find ur_e_description)/urdf/ur3e.urdf.xacro" />
+  <xacro:ur3e_robot prefix="" joint_limited="false" transmission_hw_interface="$(arg transmission_hw_interface)" />
 </robot>
