Commit message: Added support for multiple cameras (depth_camera.xacro) Removed URDF files - the files are compiled during Sim/Real robot launch Removed multiple unused launch files Refactoring of the remaining launch files

File: ur3_description/urdf/ur3_multicam.xacro (robot description, xacro)
@@ -3,7 +3,53 @@
   xmlns:xacro="http://www.ros.org/wiki/xacro">
   <xacro:include filename="$(find ur3_description)/urdf/ur3_robot_custom.urdf.xacro" />
-  <xacro:include filename="$(find ur3_description)/urdf/depth_camera.xacro" />
-  <depth_camera name="camera" />
-  <depth_camera name="camera2" />
+  <xacro:include filename="$(find ur3_description)/urdf/d435_camera_custom.urdf.xacro" />
+  <gazebo reference="camera_color_frame">
+    <sensor name="camera" type="depth">
+      <update_rate>20</update_rate>
+      <camera>
+        <horizontal_fov>1.047198</horizontal_fov>
+        <image>
+          <width>640</width>
+          <height>480</height>
+          <format>R8G8B8</format>
+        </image>
+        <clip>
+          <near>0.05</near>
+          <far>3</far>
+        </clip>
+      </camera>
+      <plugin name="camera_plugin" filename="libgazebo_ros_openni_kinect.so">
+        <baseline>0</baseline>
+        <alwaysOn>true</alwaysOn>
+        <!-- Keep this zero, update_rate in the parent <sensor> tag will control the frame rate. -->
+        <updateRate>0.0</updateRate>
+        <cameraName>camera_ir</cameraName>
+        <imageTopicName>/camera/color/image_raw</imageTopicName>
+        <cameraInfoTopicName>/camera/color/camera_info</cameraInfoTopicName>
+        <depthImageTopicName>/camera/depth/image_raw</depthImageTopicName>
+        <depthImageCameraInfoTopicName>/camera/depth/camera_info</depthImageCameraInfoTopicName>
+        <pointCloudTopicName>/camera/depth/color/points</pointCloudTopicName>
+        <frameName>camera_color_optical_frame</frameName>
+        <pointCloudCutoff>0.001</pointCloudCutoff>
+        <pointCloudCutoffMax>1.8</pointCloudCutoffMax>
+        <distortionK1>0</distortionK1>
+        <distortionK2>0</distortionK2>
+        <distortionK3>0</distortionK3>
+        <distortionT1>0</distortionT1>
+        <distortionT2>0</distortionT2>
+        <CxPrime>0</CxPrime>
+        <Cx>0</Cx>
+        <Cy>0</Cy>
+        <focalLength>0</focalLength>
+        <hackBaseline>0</hackBaseline>
+      </plugin>
+    </sensor>
+  </gazebo>
+  <link name="cam2" />
+  <joint name="world_to_cam" type="fixed">
+    <parent link="world"/>
+    <child link="cam2"/>
+    <origin xyz="0.94 -0.165 1.16" rpy="0 ${pi/6} 0"/>
+  </joint>
   <link name="world" />
   <link name="table">
@@ -38,9 +84,4 @@
     <child link="base_link_camera"/>
     <origin xyz="0.165 0.94 0.55" rpy="0 ${pi/6} -${pi/2}"/>
-  </joint>
-  <joint name="table_to_camera2" type="fixed">
-    <parent link="table"/>
-    <child link="base_link_camera2"/>
-    <origin xyz="0.94 0.165 0.55" rpy="0 ${pi/6} -${pi}"/>
   </joint>
   <link name="force_sensor">
@@ -140,3 +181,71 @@
     <origin xyz="0 0 0.076" rpy="0 0 ${pi}"/>
   </joint>
+  <link name="camera_points_link"/>
+  <joint name="camera_points_joint" type="fixed">
+    <origin rpy="0 1.57 0" xyz="0 0 0"/>
+    <parent link="base_link_camera"/>
+    <child link="camera_points_link"/>
+  </joint>
+  <xacro:property name="top_wall_z" value="0.75" />
+  <xacro:property name="limit_wall_height" value="${top_wall_z + 0.45}" />
+  <link name="top_wall">
+    <!-- <visual>
+      <geometry>
+        <box size="0.75 0.9 0.1"/>
+      </geometry>
+      <material name="black">
+        <color rgba="0 0 0 1" />
+      </material>
+    </visual> -->
+    <collision>
+      <geometry>
+        <box size="0.75 0.9 0.1"/>
+      </geometry>
+    </collision>
+  </link>
+  <joint name="top_wall_joint" type="fixed">
+    <origin rpy="0 0 0" xyz="0.2 0.18 ${top_wall_z}"/>
+    <parent link="table"/>
+    <child link="top_wall"/>
+  </joint>
+    <link name="back_wall">
+    <!-- <visual>
+      <geometry>
+        <box size="0.75 0.1 ${limit_wall_height}"/>
+      </geometry>
+      <material name="black">
+        <color rgba="0 0 0 1" />
+      </material>
+    </visual> -->
+    <collision>
+      <geometry>
+         <box size="0.75 0.1 ${limit_wall_height}"/>
+      </geometry>
+    </collision>
+  </link>
+  <joint name="back_wall_joint" type="fixed">
+    <origin rpy="0 0 0" xyz="0.2 -0.32 0.1"/>
+    <parent link="table"/>
+    <child link="back_wall"/>
+  </joint>
+    <link name="left_wall">
+    <!-- <visual>
+      <geometry>
+        <box size="0.1 0.9 ${limit_wall_height}"/>
+      </geometry>
+      <material name="black">
+        <color rgba="0 0 0 1" />
+      </material>
+    </visual> -->
+    <collision>
+      <geometry>
+         <box size="0.1 0.9 ${limit_wall_height}"/>
+      </geometry>
+    </collision>
+  </link>
+  <joint name="left_wall_joint" type="fixed">
+    <origin rpy="0 0 0" xyz="-0.22 0.18 0.1"/>
+    <parent link="table"/>
+    <child link="left_wall"/>
+  </joint>
 </robot>

Commit message: Hand tracker added

File: ur3_description/urdf/ur3_multicam.xacro (robot description, xacro)
@@ -8,3 +8,9 @@
     <origin xyz="0.94 0.165 0.55" rpy="0 ${pi/6} -${pi}"/>
   </joint>
+  <depth_camera name="camera_top" />
+  <joint name="table_to_camera_top" type="fixed">
+    <parent link="table"/>
+    <child link="base_link_camera_top"/>
+    <origin xyz="0.2 0.185 1.2" rpy="0 ${pi/2} -${pi}"/>
+  </joint>
 </robot>

Commit message: better position of top camera

File: ur3_description/urdf/ur3_multicam.xacro (robot description, xacro)
@@ -12,5 +12,5 @@
     <parent link="table"/>
     <child link="base_link_camera_top"/>
-    <origin xyz="-0.4 0.5 2.1"  rpy="0 ${pi/2} -${pi}"/>
+    <origin xyz="-0.2 0.5 2.1"  rpy="0 ${pi/2} -${pi}"/>
   </joint>
 </robot>
