Commit message: added initial version of HMI firmware

File: ur3_description/urdf/ur3_workspace_limitation.xacro (robot description, xacro)
@@ -5,6 +5,6 @@
   <xacro:property name="top_wall_z" value="0.75" />
   <xacro:property name="limit_wall_height" value="${top_wall_z + 0.45}" />
-  <link name="top_wall">
-    <!-- <visual>
+  <!--<link name="top_wall_link">
+     <visual>
       <geometry>
         <box size="0.75 0.9 0.1"/>
@@ -13,5 +13,5 @@
         <color rgba="0.2 0.2 0.2 0.2" />
       </material>
-    </visual> -->
+    </visual>
     <collision>
       <geometry>
@@ -23,7 +23,7 @@
     <origin rpy="0 0 0" xyz="0.2 0.18 ${top_wall_z}"/>
     <parent link="table"/>
-    <child link="top_wall"/>
-  </joint>
-    <link name="back_wall">
+    <child link="top_wall_link"/>
+  </joint>-->
+    <link name="back_wall_link">
     <!-- <visual>
       <geometry>
@@ -43,7 +43,7 @@
     <origin rpy="0 0 0" xyz="0.2 -0.32 0.1"/>
     <parent link="table"/>
-    <child link="back_wall"/>
+    <child link="back_wall_link"/>
   </joint>
-    <link name="left_wall">
+    <link name="left_wall_link">
     <!-- <visual>
       <geometry>
@@ -63,5 +63,5 @@
     <origin rpy="0 0 0" xyz="-0.22 0.18 0.1"/>
     <parent link="table"/>
-    <child link="left_wall"/>
+    <child link="left_wall_link"/>
   </joint>
 </robot>

Commit message: Improved positions of depth cameras Changed names of cameras and their topics

File: ur3_description/urdf/ur3_workspace_limitation.xacro (robot description, xacro)
@@ -2,5 +2,5 @@
 <robot name="ur3_workplace"
   xmlns:xacro="http://www.ros.org/wiki/xacro">
-  <xacro:include filename="$(find ur3_description)/urdf/ur3.xacro" />
+  <xacro:include filename="$(find ur3_description)/urdf/ur3e_workspace.xacro" />
   <xacro:property name="top_wall_z" value="0.75" />
   <xacro:property name="limit_wall_height" value="${top_wall_z + 0.45}" />

File: ur3_description/urdf/ur3e_workspace.xacro (robot description, xacro)
@@ -4,9 +4,21 @@
   <xacro:include filename="$(find ur3_description)/urdf/ur3_robot_custom.urdf.xacro" />
   <xacro:include filename="$(find ur3_description)/urdf/depth_camera.xacro" />
-  <depth_camera name="camera" />
-  <joint name="table_to_camera" type="fixed">
+  <depth_camera name="camera_right" />
+  <joint name="table_to_camera_right" type="fixed">
     <parent link="table"/>
-    <child link="base_link_camera"/>
-    <origin xyz="-0.4 1.4 1.6" rpy="0 ${pi/6} -${pi/2}"/>
+    <child link="base_link_camera_right"/>
+    <origin xyz="-0.6 1.2 1.6" rpy="0 ${pi/6} -${pi/4}"/>
+  </joint>
+  <depth_camera name="camera_left" />
+  <joint name="table_to_camera_left" type="fixed">
+    <parent link="table"/>
+    <child link="base_link_camera_left"/>
+    <origin xyz="-0.6 -0.2 1.6"  rpy="0 ${pi/6} ${pi/4}"/>
+  </joint>
+  <depth_camera name="camera_top" />
+  <joint name="table_to_camera_top" type="fixed">
+    <parent link="table"/>
+    <child link="base_link_camera_top"/>
+    <origin xyz="-0.2 0.5 2.1"  rpy="0 ${pi/2} -${pi}"/>
   </joint>
   <link name="world" />
