Commit message: Added adn positioned Left camera to the Real robot (UCR)

File: ur3_description/urdf/depth_camera.xacro (robot description, xacro)
@@ -2,4 +2,5 @@
 <robot name="realsense2_cameras"
     xmlns:xacro="http://ros.org/wiki/xacro">
+  <xacro:arg name="camera_range" default="1.4"/>
     <xacro:macro name="depth_camera" params="name">
         <xacro:include filename="$(find realsense2_description)/urdf/_d435.urdf.xacro" />
@@ -22,5 +23,5 @@
                         <!-- SHOULD BE EDITED ALONG WITH pointCloudCutoffMax !!! Otherwise Rviz wont start -->
                         <!-- SHOULD BE MORE THAN far_clipping_plane_distance in sensors_3d.yaml of Moveit -->
-                        <far>1.8</far>
+                        <far>$(arg camera_range)</far>
                     </clip>
                 </camera>
@@ -28,6 +29,5 @@
                     <baseline>0</baseline>
                     <alwaysOn>true</alwaysOn>
-                    <!-- Keep this zero, update_rate in the parent <sensor> tag will control the frame rate. -->
-                    <updateRate>0.0</updateRate>
+                    <updateRate>0.0</updateRate><!-- Keep this zero, update_rate in the parent <sensor> tag will control the frame rate. -->
                     <cameraName>${name}_ir</cameraName>
                     <imageTopicName>/${name}/color/image_rect_color</imageTopicName>
@@ -38,6 +38,5 @@
                     <frameName>${name}_color_optical_frame</frameName>
                     <pointCloudCutoff>0.001</pointCloudCutoff>
-                    <!-- SHOULD BE EDITED ALONG WITH clip.far !!! Otherwise Rviz wont start -->
-                    <pointCloudCutoffMax>1.8</pointCloudCutoffMax>
+                    <pointCloudCutoffMax>$(arg camera_range)</pointCloudCutoffMax>
                     <distortionK1>0</distortionK1>
                     <distortionK2>0</distortionK2>

File: ur3_description/urdf/ur3e_workspace.xacro (robot description, xacro)
@@ -4,19 +4,19 @@
   <xacro:include filename="$(find ur3_description)/urdf/ur3_robot_custom.urdf.xacro" />
   <xacro:include filename="$(find ur3_description)/urdf/depth_camera.xacro" />
-  <depth_camera name="camera_right" />
+  <!-- <depth_camera name="camera_right" />
   <joint name="table_to_camera_right" type="fixed">
     <parent link="table"/>
     <child link="base_link_camera_right"/>
     <origin xyz="-0.6 1.2 1.6" rpy="0 ${pi/6} -${pi/4}"/>
-  </joint>
+  </joint> -->
   <depth_camera name="camera_left" />
   <joint name="table_to_camera_left" type="fixed">
     <parent link="table"/>
     <child link="base_link_camera_left"/>
-    <origin xyz="-0.6 -0.2 1.6"  rpy="0 ${pi/6} ${pi/4}"/>
+    <origin xyz="-0.30 -0.26 1.71"  rpy="${-pi/2} ${pi/4} ${pi/2}"/>
   </joint>
   <depth_camera name="camera_top" />
   <joint name="table_to_camera_top" type="fixed">
-    <parent link="table"/>
+      <parent link="table"/>
     <child link="base_link_camera_top"/>
     <origin xyz="-0.22 0.47 2.0"  rpy="0 ${pi/2} -${pi}"/>
@@ -40,4 +40,29 @@
     </collision>
   </link>
+  <joint name="world_to_table" type="fixed">
+    <parent link="world"/>
+    <child link="table"/>
+    <origin xyz="0 1.0 0" rpy="0 0 -${pi}"/>
+  </joint>
+  <link name="left_wall_link">
+    <visual>
+      <geometry>
+        <box size="0.1 0.9 2.0"/>
+      </geometry>
+      <material name="black">
+        <color rgba="0.2 0.2 0.2 0.2" />
+      </material>
+    </visual>
+    <collision>
+      <geometry>
+         <box size="0.1 0.9 2.0"/>
+      </geometry>
+    </collision>
+  </link>
+  <joint name="left_wall_joint" type="fixed">
+    <origin rpy="0 0 0" xyz="2.0 0.0 0.0"/>
+    <parent link="world"/>
+    <child link="left_wall_link"/>
+  </joint>
   <link name="table_left_sup">
     <collision>
@@ -78,9 +103,4 @@
     <child link="table_back_sup"/>
     <origin xyz="0 0 0" rpy="0 0 0"/>
-  </joint>
-  <joint name="world_to_table" type="fixed">
-    <parent link="world"/>
-    <child link="table"/>
-    <origin xyz="0 1.0 0" rpy="0 0 -${pi}"/>
   </joint>
   <joint name="table_to_robot" type="fixed">
