Commit message: Updated real robot launch to utilize UR modern driver Changed urdf and goal positions definitions to fit the position of real robot Added absolute calibration from UCR robot

File: ur3_description/urdf/ur3e_workspace.xacro (robot description, xacro)
@@ -87,5 +87,5 @@
     <parent link="table"/>
     <child link="base_link"/>
-    <origin xyz="-0.58 0.49 0.972" rpy="0 0 0"/>
+    <origin xyz="-0.58 0.49 0.972" rpy="0 0 -1.57"/>
   </joint>
   <link name="force_sensor">

Commit message: Moved camera to fit the real workspace Added deifinition of real camera to launch file Added clip distance to the Real Depth camera (requires fix to the rs_rgbd.launch) Fixed ROS Camera Frame lookup timout by setting shape_transform_cache_lookup_wait_time in planning context

File: ur3_description/urdf/ur3e_workspace.xacro (robot description, xacro)
@@ -20,5 +20,5 @@
     <parent link="table"/>
     <child link="base_link_camera_top"/>
-    <origin xyz="-0.2 0.5 2.1"  rpy="0 ${pi/2} -${pi}"/>
+    <origin xyz="-0.22 0.47 2.0"  rpy="0 ${pi/2} -${pi}"/>
   </joint>
   <link name="world" />
@@ -136,5 +136,4 @@
       <geometry>
         <mesh filename="package://ur3_description/meshes/jaw.stl" scale="0.001 0.001 0.001"/>
-        <!-- <box size="0.03 0.03 0.045"/> -->
       </geometry>
       <origin rpy="${pi} 0 ${pi/2}" xyz="0 0 0"/>
@@ -153,5 +152,4 @@
     <collision>
       <geometry>
-        <!-- <box size="0.03 0.03 0.045"/> -->
         <mesh filename="package://ur3_description/meshes/jaw.stl" scale="0.001 0.001 0.001"/>
       </geometry>
@@ -169,16 +167,10 @@
     <origin xyz="0 0 0.035" rpy="0 0 0"/>
   </joint>
-  <!--<joint name="leftjaw_to_effector" type="prismatic">-->
   <joint name="leftjaw_to_effector" type="fixed">
-    <!--  <axis xyz="0 1 0"/>
-  <limit effort="1000.0" lower="0.01" upper="0" velocity="0.5"/>-->
     <parent link="effector_body"/>
     <child link="left_jaw"/>
     <origin xyz="0 0 0.076" rpy="0 0 0"/>
   </joint>
-  <!--<joint name="rightjaw_to_effector" type="prismatic">-->
   <joint name="rightjaw_to_effector" type="fixed">
-    <!--  <axis xyz="0 1 0"/>
-  <limit effort="1000.0" lower="0.01" upper="0" velocity="0.5"/> -->
     <parent link="effector_body"/>
     <child link="right_jaw"/>

Commit message: created custom gazebo settings (world) Changed workspace position to match World CS position

File: ur3_description/urdf/ur3e_workspace.xacro (robot description, xacro)
@@ -82,5 +82,5 @@
     <parent link="world"/>
     <child link="table"/>
-    <origin xyz="1 0 0" rpy="0 0 0"/>
+    <origin xyz="0 1.0 0" rpy="0 0 -${pi}"/>
   </joint>
   <joint name="table_to_robot" type="fixed">

Commit message: updated allowed collisions matrix

File: ur3_description/urdf/ur3e_workspace.xacro (robot description, xacro)
@@ -4,10 +4,10 @@
   <xacro:include filename="$(find ur3_description)/urdf/ur3_robot_custom.urdf.xacro" />
   <xacro:include filename="$(find ur3_description)/urdf/depth_camera.xacro" />
-  <!-- <depth_camera name="camera_right" />
-  <joint name="table_to_camera_right" type="fixed">
-    <parent link="table"/>
-    <child link="base_link_camera_right"/>
-    <origin xyz="-0.6 1.2 1.6" rpy="0 ${pi/6} -${pi/4}"/>
-  </joint> -->
+  <depth_camera name="camera_top" />
+  <joint name="table_to_camera_top" type="fixed">
+      <parent link="table"/>
+    <child link="base_link_camera_top"/>
+    <origin xyz="-0.22 0.47 2.0"  rpy="0 ${pi/2} -${pi}"/>
+  </joint>
   <depth_camera name="camera_left" />
   <joint name="table_to_camera_left" type="fixed">
@@ -16,9 +16,9 @@
     <origin xyz="-0.30 -0.26 1.71"  rpy="${-pi/2} ${pi/4} ${pi/2}"/>
   </joint>
-  <depth_camera name="camera_top" />
-  <joint name="table_to_camera_top" type="fixed">
-      <parent link="table"/>
-    <child link="base_link_camera_top"/>
-    <origin xyz="-0.22 0.47 2.0"  rpy="0 ${pi/2} -${pi}"/>
+  <depth_camera name="camera_right" />
+  <joint name="table_to_camera_right" type="fixed">
+    <parent link="table"/>
+    <child link="base_link_camera_right"/>
+    <origin xyz="-0.33 1.25 1.84" rpy="${-pi/2} ${pi/4} ${-pi/2}"/>
   </joint>
   <link name="world" />
@@ -44,24 +44,4 @@
     <child link="table"/>
     <origin xyz="0 1.0 0" rpy="0 0 -${pi}"/>
-  </joint>
-  <link name="left_wall_link">
-    <visual>
-      <geometry>
-        <box size="0.1 0.9 2.0"/>
-      </geometry>
-      <material name="black">
-        <color rgba="0.2 0.2 0.2 0.2" />
-      </material>
-    </visual>
-    <collision>
-      <geometry>
-         <box size="0.1 0.9 2.0"/>
-      </geometry>
-    </collision>
-  </link>
-  <joint name="left_wall_joint" type="fixed">
-    <origin rpy="0 0 0" xyz="2.0 0.0 0.0"/>
-    <parent link="world"/>
-    <child link="left_wall_link"/>
   </joint>
   <link name="table_left_sup">
@@ -109,5 +89,5 @@
     <origin xyz="-0.58 0.49 0.972" rpy="0 0 -1.57"/>
   </joint>
-  <link name="force_sensor">
+  <!-- <link name="force_sensor">
     <visual>
       <geometry>
@@ -131,6 +111,6 @@
         <mesh filename="package://ur3_description/meshes/effector_body.stl" scale="0.001 0.001 0.001"/>
       </geometry>
-      <material name="red">
-        <color rgba="1 0 0 1" />
+      <material name="gray">
+        <color rgba="0.5 0.5 0.5 1" />
       </material>
       <origin rpy="${pi/2} 0 0" xyz="0 0 0"/>
@@ -196,4 +176,4 @@
     <child link="right_jaw"/>
     <origin xyz="0 0 0.076" rpy="0 0 ${pi}"/>
-  </joint>
+  </joint> -->
 </robot>
