Commit message: Fixed fix

File: fixes/realsense-ros/realsense2_description/urdf/_materials.urdf.xacro (robot description, xacro)
@@ -9,4 +9,7 @@
   <!-- <material name="aluminum">
     <color rgba="0.5 0.5 0.5 1"/>
+  </material>
+  <material name="plastic">
+    <color rgba="0.1 0.1 0.1 1"/>
   </material> -->
 </robot>
